Commit message: MOST of part A is done! just need to finish second launch file

File: nuturtle_description/urdf/turtlebot3_burger.urdf.xacro (robot description, xacro)
@@ -3,5 +3,9 @@
   xmlns:xacro="http://ros.org/wiki/xacro">
   <!-- <xacro:include filename="$(find turtlebot3_description)/urdf/common_properties.urdf"/> -->
+  <xacro:property name="color" value="$(arg color)"/>
   <!-- Init colour -->
+  <material name="purple">
+    <color rgba="0.3 0.16 0.52 1.0"/>
+  </material>
   <material name="black">
       <color rgba="0.0 0.0 0.0 1.0"/>
@@ -46,5 +50,5 @@
         <mesh filename="package://nuturtle_description/meshes/burger_base.stl" scale="0.001 0.001 0.001"/>
       </geometry>
-      <material name="light_black"/>
+      <material name="${color}"/>
     </visual>
     <collision>

Commit message: Finished tasks A1-A5 only A6 Readme work remaining for task A

File: nuturtle_description/urdf/turtlebot3_burger.urdf.xacro (robot description, xacro)
@@ -4,4 +4,7 @@
   <!-- <xacro:include filename="$(find turtlebot3_description)/urdf/common_properties.urdf"/> -->
   <xacro:property name="color" value="$(arg color)"/>
+  <xacro:property name="yaml_file" value="$(find nuturtle_description)/config/diff_params.yaml"/>
+  <xacro:property name="ros_params" value="${xacro.load_yaml(yaml_file)['/**']}"/>
+  <xacro:property name="props" value="${ros_params['ros__parameters']}"/>
   <!-- Init colour -->
   <material name="purple">
@@ -55,5 +58,10 @@
       <origin xyz="-0.032 0 0.070" rpy="0 0 0"/>
       <geometry>
-        <box size="0.140 0.140 0.143"/>
+        <xacro:if value="${(props['collision_radius'])&gt;0}">
+          <cylinder radius="${props['wheel_radius']}" length="0.081"/>
+        </xacro:if>
+        <xacro:if value="${(props['collision_radius'])&lt;0}">
+          <box size="0.140 0.140 0.143"/>
+        </xacro:if>
       </geometry>
     </collision>
@@ -67,5 +75,5 @@
     <parent link="base_link"/>
     <child link="wheel_left_link"/>
-    <origin xyz="0.0 0.08 0.023" rpy="-1.57 0 0"/>
+    <origin xyz="0.0 ${(props['track_width'])/2} 0.023" rpy="-1.57 0 0"/>
     <axis xyz="0 0 1"/>
   </joint>
@@ -81,5 +89,5 @@
       <origin xyz="0 0 0" rpy="0 0 0"/>
       <geometry>
-        <cylinder length="0.018" radius="0.033"/>
+        <cylinder length="0.018" radius="${props['wheel_radius']}"/>
       </geometry>
     </collision>
@@ -93,5 +101,5 @@
     <parent link="base_link"/>
     <child link="wheel_right_link"/>
-    <origin xyz="0.0 -0.080 0.023" rpy="-1.57 0 0"/>
+    <origin xyz="0.0 ${-(props['track_width'])/2} 0.023" rpy="-1.57 0 0"/>
     <axis xyz="0 0 1"/>
   </joint>
@@ -107,5 +115,5 @@
       <origin xyz="0 0 0" rpy="0 0 0"/>
       <geometry>
-        <cylinder length="0.018" radius="0.033"/>
+        <cylinder length="0.018" radius="${props['wheel_radius']}"/>
       </geometry>
     </collision>
